File: KiCad/Voltage Blaster/Voltage Blaster.kicad_pcb (KiCad board)
At the start: 2 copper layers, 85.3 x 29.6 mm, 16 parts, among them J1 Bus_ISA_8bit_AB_Rev0, U1 MC79M05

Commit message: update silkscreen
Other:
- board text added: "Rear of PC ->"
Changed lines of the file:
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@@
     (property "ki_keywords" "LED diode")
     (attr through_hole)
-    (fp_text reference "D1" (at 1.275 4.445 180 unlocked) (layer "F.SilkS")
-        (effects (font (size 1 1) (thickness 0.15)))
-    )
-    (fp_text value "+5V" (at 1.296 -4.318 180 unlocked) (layer "F.SilkS")
+    (fp_text reference "D1" (at 1.275 4.445 unlocked) (layer "F.SilkS")
+        (effects (font (size 1 1) (thickness 0.15)))
+    )
+    (fp_text value "+5V" (at 1.296 -4.318 unlocked) (layer "F.SilkS")
         (effects (font (size 1 1) (thickness 0.15)))
     )
@@
     (property "ki_keywords" "R res resistor")
     (attr through_hole)
-    (fp_text reference "R1" (at 5.08 -2.37 180 unlocked) (layer "F.SilkS")
-        (effects (font (size 1 1) (thickness 0.15)))
-    )
-    (fp_text value "330R" (at 5.08 2.37 180 unlocked) (layer "F.SilkS")
+    (fp_text reference "R1" (at 5.08 -2.37 unlocked) (layer "F.SilkS")
+        (effects (font (size 1 1) (thickness 0.15)))
+    )
+    (fp_text value "330R" (at 5.08 2.37 unlocked) (layer "F.SilkS")
         (effects (font (size 1 1) (thickness 0.15)))
     )
@@
         (effects (font (size 1 1) (thickness 0.15)))
     )
-    (fp_text value "MC79M05" (at 0 4.5 180 unlocked) (layer "F.SilkS")
+    (fp_text value "MC79M05" (at 0 4.5 unlocked) (layer "F.SilkS")
         (effects (font (size 1 1) (thickness 0.15)))
     )
@@
     (property "ki_keywords" "R res resistor")
     (attr through_hole)
-    (fp_text reference "R4" (at 5.08 -2.37 180 unlocked) (layer "F.SilkS")
-        (effects (font (size 1 1) (thickness 0.15)))
-    )
-    (fp_text value "1K" (at 5.08 2.37 180 unlocked) (layer "F.SilkS")
+    (fp_text reference "R4" (at 5.08 -2.37 unlocked) (layer "F.SilkS")
+        (effects (font (size 1 1) (thickness 0.15)))
+    )
+    (fp_text value "1K" (at 5.08 2.37 unlocked) (layer "F.SilkS")
         (effects (font (size 1 1) (thickness 0.15)))
     )
@@
     (property "ki_keywords" "R res resistor")
     (attr through_hole)
-    (fp_text reference "R3" (at 5.08 -2.37 180 unlocked) (layer "F.SilkS")
-        (effects (font (size 1 1) (thickness 0.15)))
-    )
-    (fp_text value "330R" (at 5.053 2.388 180 unlocked) (layer "F.SilkS")
+    (fp_text reference "R3" (at 5.08 -2.37 unlocked) (layer "F.SilkS")
+        (effects (font (size 1 1) (thickness 0.15)))
+    )
+    (fp_text value "330R" (at 5.053 2.388 unlocked) (layer "F.SilkS")
         (effects (font (size 1 1) (thickness 0.15)))
     )
@@
     (property "ki_keywords" "LED diode")
     (attr through_hole)
-    (fp_text reference "D2" (at 1.2192 4.445 180 unlocked) (layer "F.SilkS")
-        (effects (font (size 1 1) (thickness 0.15)))
-    )
-    (fp_text value "+12V" (at 1.416 -4.318 180 unlocked) (layer "F.SilkS")
+    (fp_text reference "D2" (at 1.2192 4.445 unlocked) (layer "F.SilkS")
+        (effects (font (size 1 1) (thickness 0.15)))
+    )
+    (fp_text value "+12V" (at 1.3474 -4.3176 unlocked) (layer "F.SilkS")
         (effects (font (size 1 1) (thickness 0.15)))
     )
@@
     (property "ki_keywords" "LED diode")
     (attr through_hole)
-    (fp_text reference "D4" (at 1.402 4.445 180 unlocked) (layer "F.SilkS")
-        (effects (font (size 1 1) (thickness 0.15)))
-    )
-    (fp_text value "-12V" (at 1.529 -4.318 180 unlocked) (layer "F.SilkS")
+    (fp_text reference "D4" (at 1.402 4.445 unlocked) (layer "F.SilkS")
+        (effects (font (size 1 1) (thickness 0.15)))
+    )
+    (fp_text value "-12V" (at 1.2384 -4.3076 unlocked) (layer "F.SilkS")
         (effects (font (size 1 1) (thickness 0.15)))
     )
@@
     (property "ki_keywords" "R res resistor")
     (attr through_hole)
-    (fp_text reference "R2" (at 5.08 -2.37 180 unlocked) (layer "F.SilkS")
-        (effects (font (size 1 1) (thickness 0.15)))
-    )
-    (fp_text value "1K" (at 5.042 2.408 180 unlocked) (layer "F.SilkS")
+    (fp_text reference "R2" (at 5.08 -2.37 unlocked) (layer "F.SilkS")
+        (effects (font (size 1 1) (thickness 0.15)))
+    )
+    (fp_text value "1K" (at 5.042 2.408 unlocked) (layer "F.SilkS")
         (effects (font (size 1 1) (thickness 0.15)))
     )
@@
     (property "ki_keywords" "Jumper SPST")
     (attr through_hole)
-    (fp_text reference "JP1" (at 2.4384 1.2192 180 unlocked) (layer "F.SilkS")
+    (fp_text reference "JP1" (at 2.4384 1.2192 unlocked) (layer "F.SilkS")
         (effects (font (size 1 1) (thickness 0.15)))
     )
@@
     (property "ki_keywords" "cap capacitor")
     (attr through_hole)
-    (fp_text reference "C2" (at 1 -3.75 180 unlocked) (layer "F.SilkS")
-        (effects (font (size 1 1) (thickness 0.15)))
-    )
-    (fp_text value "22uF" (at 1 3.75 180 unlocked) (layer "F.SilkS")
+    (fp_text reference "C2" (at 1 -3.75 unlocked) (layer "F.SilkS")
+        (effects (font (size 1 1) (thickness 0.15)))
+    )
+    (fp_text value "22uF" (at 1 3.75 unlocked) (layer "F.SilkS")
         (effects (font (size 1 1) (thickness 0.15)))
     )
@@
     (property "ki_keywords" "diode")
     (attr through_hole)
-    (fp_text reference "D6" (at 3.81 -2.47 180 unlocked) (layer "F.SilkS")
-        (effects (font (size 1 1) (thickness 0.15)))
-    )
-    (fp_text value "SB140" (at 3.81 2.47 180 unlocked) (layer "F.SilkS")
+    (fp_text reference "D6" (at 3.81 -2.47 unlocked) (layer "F.SilkS")
+        (effects (font (size 1 1) (thickness 0.15)))
+    )
+    (fp_text value "SB140" (at 3.81 2.47 unlocked) (layer "F.SilkS")
         (effects (font (size 1 1) (thickness 0.15)))
     )
@@
     (property "ki_keywords" "LED diode")
     (attr through_hole)
-    (fp_text reference "D3" (at 1.409 4.445 180 unlocked) (layer "F.SilkS")
-        (effects (font (size 1 1) (thickness 0.15)))
-    )
-    (fp_text value "-5V" (at 1.663 -4.318 180 unlocked) (layer "F.SilkS")
+    (fp_text reference "D3" (at 1.409 4.445 unlocked) (layer "F.SilkS")
+        (effects (font (size 1 1) (thickness 0.15)))
+    )
+    (fp_text value "-5V" (at 1.2354 -4.3076 unlocked) (layer "F.SilkS")
         (effects (font (size 1 1) (thickness 0.15)))
     )
@@
     (property "ki_keywords" "diode")
     (attr through_hole)
-    (fp_text reference "D5" (at 3.81 -2.47 180 unlocked) (layer "F.SilkS")
-        (effects (font (size 1 1) (thickness 0.15)))
-    )
-    (fp_text value "SB140" (at 3.81 2.47 180 unlocked) (layer "F.SilkS")
+    (fp_text reference "D5" (at 3.81 -2.47 unlocked) (layer "F.SilkS")
+        (effects (font (size 1 1) (thickness 0.15)))
+    )
+    (fp_text value "SB140" (at 3.81 2.47 unlocked) (layer "F.SilkS")
         (effects (font (size 1 1) (thickness 0.15)))
     )
@@
     (property "ki_keywords" "cap capacitor")
     (attr through_hole)
-    (fp_text reference "C1" (at 1 -3.75 180 unlocked) (layer "F.SilkS")
-        (effects (font (size 1 1) (thickness 0.15)))
-    )
-    (fp_text value "22uF" (at 1 3.75 180 unlocked) (layer "F.SilkS")
+    (fp_text reference "C1" (at 1 -3.75 unlocked) (layer "F.SilkS")
+        (effects (font (size 1 1) (thickness 0.15)))
+    )
+    (fp_text value "22uF" (at 1 3.75 unlocked) (layer "F.SilkS")
         (effects (font (size 1 1) (thickness 0.15)))
     )
@@
     (effects (font (size 1 1) (thickness 0.15)) (justify left bottom mirror))
   )
-  (gr_text "<- Rear of PC" (at 199.644 92.075 180) (layer "F.SilkS")
+  (gr_text "Rear of PC ->" (at 182.06 93.6) (layer "F.SilkS")
     (effects (font (size 1.5 1.5) (thickness 0.2) bold) (justify left bottom))
   )
-  (gr_text "JP1:\nOutput\nDisconnect" (at 197.4088 94.996 180) (layer "F.SilkS")
+  (gr_text "JP1:\nOutput\nDisconnect" (at 189.2 99.83) (layer "F.SilkS")
     (effects (font (size 0.8 0.8) (thickness 0.1)) (justify left bottom))
   )
-  (gr_text "Voltage Blaster\n(Enhanced)" (at 161.29 99.3648 180) (layer "F.SilkS")
+  (gr_text "Voltage Blaster\n(Enhanced)" (at 161.21 102.03) (layer "F.SilkS")
     (effects (font (size 1.25 1.25) (thickness 0.3) bold) (justify bottom))
   )
-  (gr_text "Protection\nDiodes" (at 187.325 110.236 180) (layer "F.SilkS")
+  (gr_text "Protection\nDiodes" (at 187.325 110.236) (layer "F.SilkS")
     (effects (font (size 0.8 0.8) (thickness 0.15)))
   )
